File: hardware/main.brd (EAGLE design)
At the start: 62.2 x 75.8 mm, 28 parts, among them IC3 E73_2G4M04S, J3 DCJ0202, J4 SCREWTERMINAL_3X, Q1 BUZ11, Q2 BUZ11, Q3 BUZ11, Q4 BUZ11

Commit message: enhanced Readme after testing
Connections:
- net RX: now also J1.4; no longer J1.5
- net TX: now also J1.5; no longer J1.4
Routing:
- net TX: track 22.8 -> 27.1 mm
- net RX: track 23.5 -> 20.6 mm
Changed lines of the file:
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@@
 <drawing>
 <settings>
-<setting alwaysvectorfont="yes"/>
+<setting alwaysvectorfont="no"/>
 <setting verticaltext="up"/>
 </settings>
@@
 <vertex x="25.4" y="0"/>
 <vertex x="29.5" y="6"/>
-<vertex x="29.5" y="6"/>
 <vertex x="62.2" y="6"/>
 <vertex x="62.2" y="0"/>
@@
 <vertex x="25.4" y="0"/>
 <vertex x="29.5" y="6"/>
-<vertex x="29.5" y="6"/>
 <vertex x="62.2" y="6"/>
 <vertex x="62.2" y="0"/>
@@
 <signal name="TX">
 <contactref element="IC3" pad="21"/>
-<contactref element="J1" pad="4"/>
 <wire x1="49.925" y1="28.77" x2="49.925" y2="29.975" width="0.2032" layer="1"/>
 <wire x1="36.8" y1="33.9" x2="36.2" y2="34.5" width="0.2032" layer="1"/>
-<wire x1="36.2" y1="34.5" x2="36.2" y2="38.93" width="0.2032" layer="1"/>
-<wire x1="36.2" y1="38.93" x2="37.3" y2="40.03" width="0.2032" layer="1"/>
 <wire x1="49.925" y1="29.975" x2="46" y2="33.9" width="0.2032" layer="1"/>
 <wire x1="46" y1="33.9" x2="36.8" y2="33.9" width="0.2032" layer="1"/>
+<contactref element="J1" pad="5"/>
+<wire x1="36.9" y1="38.8" x2="38" y2="38.8" width="0.2032" layer="1"/>
+<wire x1="38" y1="38.8" x2="38.6" y2="39.4" width="0.2032" layer="1"/>
+<wire x1="38.6" y1="41.27" x2="37.3" y2="42.57" width="0.2032" layer="1"/>
+<wire x1="36.2" y1="34.5" x2="36.2" y2="38.1" width="0.2032" layer="1"/>
+<wire x1="36.2" y1="38.1" x2="36.9" y2="38.8" width="0.2032" layer="1"/>
+<wire x1="38.6" y1="39.4" x2="38.6" y2="41.27" width="0.2032" layer="1"/>
 </signal>
 <signal name="RX">
 <contactref element="IC3" pad="23"/>
-<contactref element="J1" pad="5"/>
 <wire x1="47.385" y1="28.77" x2="47.385" y2="30.1848" width="0.2032" layer="1"/>
 <wire x1="47.385" y1="30.1848" x2="44" y2="33.5698" width="0.2032" layer="1"/>
 <wire x1="44" y1="33.5698" x2="36.663225" y2="33.5698" width="0.2032" layer="1"/>
 <wire x1="36.663225" y1="33.5698" x2="35.8698" y2="34.363225" width="0.2032" layer="1"/>
-<wire x1="35.8698" y1="34.363225" x2="35.8698" y2="41.1408875" width="0.2032" layer="1"/>
-<wire x1="37.3" y1="42.57" x2="37.2989125" y2="42.57" width="0.2032" layer="1"/>
-<wire x1="37.2989125" y1="42.57" x2="35.8698" y2="41.1408875" width="0.2032" layer="1"/>
+<wire x1="35.8698" y1="34.363225" x2="35.8698" y2="38.5408875" width="0.2032" layer="1"/>
+<wire x1="37.0989125" y1="39.77" x2="35.8698" y2="38.5408875" width="0.2032" layer="1"/>
+<contactref element="J1" pad="4"/>
+<wire x1="37.0989125" y1="39.77" x2="37.3" y2="40.03" width="0" layer="19" extent="1-1"/>
 </signal>
 <signal name="+3V3">
